File: hardware/alpha_board.brd (EAGLE design)
At the start: 47 x 39.4 mm, 13 parts

Commit message: update to Alpha Kit v0.4
Parts:
- added AUDIO, AUDIO1: (no value), SparkFun:1X03_LOCK
- added C1, R7: (no value), SparkFun:1206
- added U$2: MICROSD-HIROSE, calculator_lib:MICROSD_HOLDER-HIROSE-DM3AT
- R4: value 4,7 -> (none)
- R5: value 4,7k -> (none)
- moved R4 26.9 mm to (17.8, 44.5), turned to 180 degrees
- moved R5 15.9 mm to (44.5, 21.6), turned to 90 degrees
- renumbered I2C to ADC
Connections:
- removed net A0: JP1.12
- removed net A4: JP1.8
- removed net D0(SDA): ADC.3, JP2.12, R4.1
- removed net D1(SCL): ADC.2, JP2.11, R5.1
- new net GNDB: ADC.4, AUDIO.2, AUDIO1.2, C1.1, DS18B20_EXT.3, DS18B20_INT.3, R7.2, U$2.CD1, U$2.VSS
- new net N$1: JP1.10, R4.1, U$2.DAT3
- new net N$2: AUDIO.1, JP1.12
- new net N$3: JP1.8, U$2.DAT0
- new net N$6: AUDIO1.1, JP1.11
- new net VCCB: ADC.1, AUDIO.3, AUDIO1.3, R5.2
- net A3: now also U$2.CLK
- net A5: now also U$2.CMD
- net D6: now also ADC.3
- net D7: now also ADC.2
- net GND: now also R7.1; no longer ADC.4, DS18B20_EXT.3, DS18B20_INT.3
- net VCC: now also C1.2, R5.1, U$2.VDD; no longer ADC.1, R5.2
Routing:
- net GNDB: track 0.00 -> 145.9 mm
- net VCCB: track 0.00 -> 44.2 mm
- net D7: track 0.00 -> 34.1 mm
- net GND: track 63.3 -> 32.7 mm
- net D6: track 0.00 -> 30.0 mm
- net N$1: track 0.00 -> 28.6 mm
- net A3: track 0.00 -> 24.3 mm
- net N$3: track 0.00 -> 21.5 mm
- net D1(SCL): track 21.0 -> 0.00 mm
- net D0(SDA): track 16.2 -> 0.00 mm
- net A5: track 0.00 -> 14.9 mm
- net N$6: track 0.00 -> 13.7 mm
- net VCC: track 164.5 -> 158.2 mm
- net N$2: track 0.00 -> 5.34 mm
- added copper zone on layer 1, net GNDB
- removed copper zone on layer 1, net GND
Other:
- board size 47 x 39.4 mm -> 47 x 58.6 mm
