File: hardware/alpha_board.sch (EAGLE design)
At the start: 13 parts

Commit message: update to Alpha Kit v0.4
Parts:
- added AUDIO, AUDIO1: (no value), SparkFun:M03LOCK
- added C1: (no value), SparkFun:CAP1206
- added R7: (no value), SparkFun:RESISTOR1206
- added U$2: MICROSD-HIROSE, calculator_lib:MICROSD-HIROSE
- R4: value 4,7 -> (none)
- R5: value 4,7k -> (none)
- renumbered I2C to ADC
Connections:
- removed net A0: JP1.12
- removed net A4: JP1.8
- removed net D0(SDA): ADC.3, JP2.12, R4.1
- removed net D1(SCL): ADC.2, JP2.11, R5.1
- new net GNDB: ADC.4, AUDIO.2, AUDIO1.2, C1.1, DS18B20_EXT.3, DS18B20_INT.3, R7.2, U$2.CD1, U$2.GND
- new net N$1: JP1.10, R4.1, U$2.CS
- new net N$2: AUDIO.1, JP1.12
- new net N$3: JP1.8, U$2.DO
- new net N$6: AUDIO1.1, JP1.11
- new net VCCB: ADC.1, AUDIO.3, AUDIO1.3, R5.2
- net A3: now also U$2.SCK
- net A5: now also U$2.DI
- net D6: now also ADC.3
- net D7: now also ADC.2
- net GND: now also R7.1; no longer ADC.4, DS18B20_EXT.3, DS18B20_INT.3
- net VCC: now also C1.2, R5.1, U$2.VCC; no longer ADC.1, R5.2
Other:
- moved on the sheet: R4, R5
